File: IoT_Node.kicad_pcb (KiCad board)
At the start: 2 copper layers, 103 x 86.5 mm, 69 parts, among them J1 Conn_01x03, J10 IOT2Connector_Int, J2 Conn_01x03, J3 Conn_01x03, J4 Conn_01x03, J5 Conn_01x03, J6 Conn_01x03, J7 RJ45-TRANSFO, J8 Conn_01x03, J9 Conn_01x03, U1 ICSP6, U10 Relay, U11 1N4148, U12 Relay, U13 MOSFET, U14 MOSFET, U15 1N4148, U16 Relay, U17 1N4148, U18 Relay, U19 ENC28J60-C/SS, U2 ESP-12E, U20 LM2575, U21 Button, U3 ICSP6, U4 Button, U5 ATMEGA324A-AU, U6 IOT2Connector, U7 MOSFET, U8 MOSFET, U9 1N4148, Y1 10MHz, Y2 25MHz

Commit message: board erweitert
Parts:
- turned C10 to 0 degrees
Routing:
- net GND: track 31.1 -> 385.3 mm
- net +3V3: track 0.00 -> 243.1 mm, vias 0 -> 6
- net +12V: track 29.8 -> 170.9 mm
- net /IO4: track 0.00 -> 98.0 mm, vias 0 -> 3
- net /IO6: track 0.00 -> 86.5 mm, vias 0 -> 2
- net /IO5: track 0.00 -> 80.0 mm, vias 0 -> 2
- net /ADC0: track 0.00 -> 68.6 mm, vias 0 -> 1
- net /1wire: track 0.00 -> 55.7 mm, vias 0 -> 2
- net /MISO2: track 0.00 -> 54.2 mm, vias 0 -> 2
- net Net-(U11-Pad1): track 10.9 -> 50.6 mm
- net Net-(J5-Pad2): track 0.00 -> 39.1 mm
- net Net-(J3-Pad2): track 0.00 -> 38.9 mm
- net /enc28j60/TPIN+: track 0.00 -> 38.8 mm
- net /MOSI2: track 0.00 -> 37.4 mm, vias 0 -> 2
- net /ETH_CS: track 0.00 -> 36.9 mm, vias 0 -> 2
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
Commit message: erste Funktionierende Version
Parts:
- added REF**: MountingHole_3.2mm_M3, Mounting_Holes:MountingHole_3.2mm_M3, F.Cu at (39.0, 98.0)
- added REF**: MountingHole_3.2mm_M3, Mounting_Holes:MountingHole_3.2mm_M3, F.Cu at (124.0, 48.0)
- moved C3 18.6 mm to (78.5, 63.6), turned to 45 degrees
- moved C15 17.3 mm to (91.7, 55.2)
- moved U3 14.6 mm to (92.2, 79.9), turned to 270 degrees
- moved J1 11.7 mm to (94.1, 91.2)
- moved J2 11.7 mm to (90.0, 91.2)
- moved C2 8.36 mm to (85.3, 70.5), turned to 45 degrees
- moved Y1 6.99 mm to (79.9, 72.5), turned to 135 degrees
- moved C11 6.63 mm to (65.3, 85.0), turned to 315 degrees
- moved C9 5.74 mm to (53.2, 87.2), turned to 90 degrees
- moved C12 4.06 mm to (67.3, 63.2)
- moved U5 3.64 mm to (71.9, 79.0), turned to 225 degrees
- moved C1 3.30 mm to (67.3, 61.0)
- moved C8 2.79 mm to (67.3, 58.7)
- moved C14 2.67 mm to (77.9, 85.5), turned to 45 degrees
- moved C10 2.29 mm to (67.3, 56.4)
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Routing:
- net /IO1: track 13.4 -> 208.5 mm, vias 0 -> 6
- net GND: track 385.3 -> 570.2 mm, vias 0 -> 15
- net /IO0: track 15.6 -> 187.8 mm, vias 0 -> 5
- net +12V: track 170.9 -> 309.3 mm, vias 0 -> 4
- net +3V3: track 243.1 -> 377.9 mm, vias 6 -> 5
- net /IO3: track 9.96 -> 123.7 mm, vias 0 -> 5
- net /IO2: track 13.4 -> 116.9 mm, vias 0 -> 4
- net /RXD: track 9.09 -> 107.3 mm, vias 0 -> 3
- net /TXD: track 9.09 -> 100.8 mm, vias 0 -> 2
- net /I2C_SCL: track 10.3 -> 92.9 mm, vias 0 -> 2
- net /I2C_SDA: track 10.4 -> 91.4 mm, vias 0 -> 2
- net /ESP_BOOT: track 0.00 -> 55.5 mm, vias 0 -> 4
- net /RST1: track 0.00 -> 52.8 mm, vias 0 -> 2
- net /IO7: track 6.55 -> 56.3 mm, vias 0 -> 5
- net /MOSI1: track 26.4 -> 74.9 mm, vias 2 -> 3
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- added copper zone on B.Cu, net GND
- added copper zone on F.Cu, net GND
Other:
- outline, holes or cut-outs redrawn
- board text added: "3,3V MOSI GND"
- board text added: "MISO SCK RST"
