File: IoT_Node.sch (KiCad schematic (older format))
At the start: 33 parts, among them J1 Conn_01x03, J10 IOT2Connector_Int, J2 Conn_01x03, J8 Conn_01x03, J9 Conn_01x03, U1 ICSP6, U2 ESP-12E, U20 LM2575, U3 ICSP6, U4 Button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

Commit message: erste Funktionierende Version
Parts:
- gave numbers to parts that had none: 1
